File: eagle/tutorial/msl.brd (EAGLE design)
At the start: 20 x 20 mm, 5 parts

Commit message: tutorial
Routing:
- net V2: track 7.35 -> 0.00 mm
- net V1: track 7.35 -> 0.00 mm
- added copper zone on layer 1, net V1
- added copper zone on layer 1, net V2
Changed lines of the file:
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@@
 <contactref element="TP1" pad="TP"/>
 <contactref element="C1" pad="1"/>
-<wire x1="9.35" y1="10" x2="2" y2="10" width="0.1016" layer="1"/>
+<polygon width="0" layer="1" thermals="no">
+<vertex x="1.95" y="10.0508"/>
+<vertex x="9.8" y="10.0508"/>
+<vertex x="9.8" y="9.9492"/>
+<vertex x="1.95" y="9.9492"/>
+</polygon>
 </signal>
 <signal name="V2">
 <contactref element="C1" pad="2"/>
 <contactref element="TP2" pad="TP"/>
-<wire x1="18" y1="10" x2="10.65" y2="10" width="0.1016" layer="1"/>
+<polygon width="0" layer="1" thermals="no">
+<vertex x="10.2" y="10.0508"/>
+<vertex x="18.05" y="10.0508"/>
+<vertex x="18.05" y="9.9492"/>
+<vertex x="10.2" y="9.9492"/>
+</polygon>
 </signal>
 <signal name="GND">
